File: v0.4/Interface boards/Jeep JTEC/ccd_decoder.sch (KiCad schematic (older format))
At the start: 19 parts, among them Q1 AO3400, Q2 IRF7317, U1 LM2903, U2 USBLC6-2SC6

Commit message: Correct drill size for JTEC connector
Parts:
- JP1, JP2: Manufacturer 10129378-902001BLF -> Amphenol ICC (FCI); Manufacturer# Amphenol ICC (FCI) -> 10129378-902001BLF
Changed lines of the file:
@@
 F 2 "Connector_PinHeader_2.54mm:PinHeader_1x02_P2.54mm_Vertical" H 10250 1700 50  0001 C CNN
 F 3 "~" H 10250 1700 50  0001 C CNN
-F 4 "10129378-902001BLF" H 10250 1700 50  0001 C CNN "Manufacturer"
-F 5 "Amphenol ICC (FCI)" H 10250 1700 50  0001 C CNN "Manufacturer#"
+F 4 "Amphenol ICC (FCI)" H 10250 1700 50  0001 C CNN "Manufacturer"
+F 5 "10129378-902001BLF" H 10250 1700 50  0001 C CNN "Manufacturer#"
 F 6 "10129378-902001BLF-ND" H 10250 1700 50  0001 C CNN "digikey#"
 	1    10250 1700
@@
 F 2 "Connector_PinHeader_2.54mm:PinHeader_1x02_P2.54mm_Vertical" H 10250 2200 50  0001 C CNN
 F 3 "~" H 10250 2200 50  0001 C CNN
-F 4 "10129378-902001BLF" H 10250 2200 50  0001 C CNN "Manufacturer"
-F 5 "Amphenol ICC (FCI)" H 10250 2200 50  0001 C CNN "Manufacturer#"
+F 4 "Amphenol ICC (FCI)" H 10250 2200 50  0001 C CNN "Manufacturer"
+F 5 "10129378-902001BLF" H 10250 2200 50  0001 C CNN "Manufacturer#"
 F 6 "10129378-902001BLF-ND" H 10250 2200 50  0001 C CNN "digikey#"
 	1    10250 2200
